File: ecad/HassRoomSensor.kicad_sch (KiCad schematic)
At the start: 31 parts, among them J1 Conn_01x04_Pin, J2 62131021021, J3 Conn_01x04_Pin, J4 Conn_01x02_Pin, U1 SCD40-D-R2, U2 BME690, U3 XIAO ESP32C6

Commit message: updated/fixed JLCPCB part numbers
Parts:
- C1, C6, C7: JLCPCB Part # CL21B106KOQNNNE -> C95841
- C2, C3, C4, C5, C8: JLCPCB Part # CL05A104KA5NNNC -> C100072
- D1: JLCPCB Part # 150060RS75000 -> C3030991
- D2: JLCPCB Part # 150060GS75000 -> C5252984
- J2: JLCPCB Part # (none) -> C21202083
- J4: JLCPCB Part # S2B-PH-SM4-TB(LF)(SN) -> C295747
- R1: JLCPCB Part # RC0603FR-07130RL -> C6823558
- R2: JLCPCB Part # RC0402FR-071RL -> C7038446
- R3: JLCPCB Part # RC0603FR-0710RL -> C723701
- R4: JLCPCB Part # SR0805FR-471RL -> C873764
- R5, R6, R8: JLCPCB Part # RC0402FR-0710KL -> C851816
- R7: JLCPCB Part # RC0402FR-078K2L -> C20161309
- U1: JLCPCB Part # (none) -> C3659421
- U2: JLCPCB Part # BME690 -> C42431867; Manufacturer (none) -> Bosch
Changed lines of the file:
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@@
 			)
 		)
-		(property "JLCPCB Part #" "CL05A104KA5NNNC"
+		(property "JLCPCB Part #" "C100072"
 			(at 107.95 127 0)
 			(effects
@@
 			)
 		)
-		(property "JLCPCB Part #" "RC0402FR-071RL"
+		(property "JLCPCB Part #" "C7038446"
 			(at 53.34 160.02 90)
 			(effects
@@
 			)
 		)
-		(property "JLCPCB Part #" "CL05A104KA5NNNC"
+		(property "JLCPCB Part #" "C100072"
 			(at 66.04 167.64 0)
 			(effects
@@
 			)
 		)
-		(property "JLCPCB Part #" "CL21B106KOQNNNE"
+		(property "JLCPCB Part #" "C95841"
 			(at 156.21 49.53 0)
 			(effects
@@
 			)
 		)
-		(property "JLCPCB Part #" "CL21B106KOQNNNE"
+		(property "JLCPCB Part #" "C95841"
 			(at 41.91 168.91 0)
 			(effects
@@
 			)
 		)
-		(property "JLCPCB Part #" ""
+		(property "JLCPCB Part #" "C3659421"
 			(at 60.96 127 0)
 			(effects
@@
 			)
 		)
-		(property "JLCPCB Part #" "CL05A104KA5NNNC"
+		(property "JLCPCB Part #" "C100072"
 			(at 246.38 52.07 0)
 			(effects
@@
 			)
 		)
-		(property "JLCPCB Part #" "150060GS75000"
+		(property "JLCPCB Part #" "C5252984"
 			(at 55.88 87.63 90)
 			(effects
@@
 			)
 		)
-		(property "JLCPCB Part #" "SR0805FR-471RL"
+		(property "JLCPCB Part #" "C873764"
 			(at 118.11 119.38 90)
 			(effects
@@
 			)
 		)
-		(property "JLCPCB Part #" "150060RS75000"
+		(property "JLCPCB Part #" "C3030991"
 			(at 38.1 87.63 90)
 			(effects
@@
 			)
 		)
-		(property "JLCPCB Part #" "RC0603FR-07130RL"
+		(property "JLCPCB Part #" "C6823558"
 			(at 38.1 78.74 90)
 			(effects
@@
 			)
 		)
-		(property "JLCPCB Part #" ""
+		(property "JLCPCB Part #" "C21202083"
 			(at 196.85 101.6 90)
 			(effects
@@
 			)
 		)
-		(property "JLCPCB Part #" "BME690"
+		(property "JLCPCB Part #" "C42431867"
+			(at 101.6 161.29 0)
+			(effects
+				(font
+					(size 1.27 1.27)
+				)
+				(hide yes)
+			)
+		)
+		(property "Manufacturer" "Bosch"
 			(at 101.6 161.29 0)
 			(effects
@@
 			)
 		)
-		(property "JLCPCB Part #" "S2B-PH-SM4-TB(LF)(SN)"
+		(property "JLCPCB Part #" "C295747"
 			(at 227.33 45.72 0)
 			(effects
@@
 			)
 		)
-		(property "JLCPCB Part #" "RC0402FR-0710KL"
+		(property "JLCPCB Part #" "C851816"
 			(at 199.39 48.26 0)
 			(effects
@@
 			)
 		)
-		(property "JLCPCB Part #" "RC0402FR-0710KL"
+		(property "JLCPCB Part #" "C851816"
 			(at 187.96 48.26 0)
 			(effects
@@
 			)
 		)
-		(property "JLCPCB Part #" "RC0402FR-0710KL"
+		(property "JLCPCB Part #" "C851816"
 			(at 238.76 52.07 0)
 			(effects
@@
 			)
 		)
-		(property "JLCPCB Part #" "CL05A104KA5NNNC"
+		(property "JLCPCB Part #" "C100072"
 			(at 76.2 167.64 0)
 			(effects
@@
 			)
 		)
-		(property "JLCPCB Part #" "CL05A104KA5NNNC"
+		(property "JLCPCB Part #" "C100072"
 			(at 91.44 127 0)
 			(effects
@@
 			)
 		)
-		(property "JLCPCB Part #" "CL21B106KOQNNNE"
+		(property "JLCPCB Part #" "C95841"
 			(at 129.54 127 0)
 			(effects
@@
 			)
 		)
-		(property "JLCPCB Part #" "RC0402FR-078K2L"
+		(property "JLCPCB Part #" "C20161309"
 			(at 238.76 41.91 0)
 			(effects
@@
 			)
 		)
-		(property "JLCPCB Part #" "RC0603FR-0710RL"
+		(property "JLCPCB Part #" "C723701"
 			(at 55.88 78.74 90)
 			(effects
